Commit message: Update: シミュレータ内ではキャスタホイールと車輪が同じ高さで接地する
シミュレーションでは傾きがLiDARのノイズの原因になっていたので，正確ではないが高さを揃えて対処した

File: adamr2_description/urdf/robot_sim.xacro (robot description, xacro)
@@ -35,5 +35,5 @@
   <!-- back -->
   <xacro:caster prefix="back" parent="base_link">
-    <origin xyz="-0.275 0.0 -0.1498"/>
+    <origin xyz="-0.275 0.0 -0.1525"/>
     <axis xyz="0 0 1"/>
   </xacro:caster>
@@ -41,5 +41,5 @@
   <!-- front -->
   <xacro:caster prefix="front" parent="base_link">
-    <origin xyz="0.275 0.0 -0.1498" rpy="0 0 ${radians(180)}"/>
+    <origin xyz="0.275 0.0 -0.1525" rpy="0 0 ${radians(180)}"/>
     <axis xyz="0 0 1"/>
   </xacro:caster>
@@ -47,5 +47,5 @@
   <!-- lidar -->
   <xacro:lidar parent="base_link">
-    <origin xyz="0.275 0 0.177" rpy="0 0 ${radians(180)}"/>
+    <origin xyz="0.275 0 0.177" rpy="0 0 0"/>
   </xacro:lidar>
   <xacro:lidar_gazebo/>
