Commit message: Fix: 各リンクのZ軸方向の距離を修正

File: adamr2_description/urdf/robot.xacro (robot description, xacro)
@@ -13,10 +13,10 @@
   <!-- left -->
   <xacro:wheel prefix="left" parent="base_link">
-    <origin xyz="0.0 0.1915 -184.5"/>
+    <origin xyz="0.0 0.1915 -0.1845"/>
     <axis xyz="0 1 0"/>
   </xacro:wheel>
   <!-- right -->
   <xacro:wheel prefix="right" parent="base_link">
-    <origin xyz="0.0 -0.1915 -184.5"/>
+    <origin xyz="0.0 -0.1915 -0.1845"/>
     <axis xyz="0 -1 0"/>
   </xacro:wheel>
@@ -24,10 +24,10 @@
   <!-- back -->
   <xacro:caster prefix="back" parent="base_link">
-    <origin xyz="-0.275 0.0 -149.8"/>
+    <origin xyz="-0.275 0.0 -0.1498"/>
     <axis xyz="0 0 1"/>
   </xacro:caster>
   <!-- front -->
   <xacro:caster prefix="front" parent="base_link">
-    <origin xyz="0.275 0.0 -149.8"/>
+    <origin xyz="0.275 0.0 -0.1498"/>
     <axis xyz="0 0 1"/>
   </xacro:caster>

Commit message: Update: 車輪の軸の向きを修正
ロボットが前に進んだときの回転方向が正になる向き

File: adamr2_description/urdf/robot.xacro (robot description, xacro)
@@ -19,5 +19,5 @@
   <xacro:wheel prefix="right" parent="base_link">
     <origin xyz="0.0 -0.1915 -0.1845"/>
-    <axis xyz="0 -1 0"/>
+    <axis xyz="0 1 0"/>
   </xacro:wheel>
   <!--casters-->
@@ -29,5 +29,5 @@
   <!-- front -->
   <xacro:caster prefix="front" parent="base_link">
-    <origin xyz="0.275 0.0 -0.1498"/>
+    <origin xyz="0.275 0.0 -0.1498" rpy="0 0 ${radians(180)}"/>
     <axis xyz="0 0 1"/>
   </xacro:caster>

Commit message: Fix: Lidarの座標系を修正した

File: adamr2_description/urdf/robot.xacro (robot description, xacro)
@@ -35,5 +35,5 @@
   <!-- lidar -->
   <xacro:lidar parent="base_link">
-    <origin xyz="0.275 0 0.177"/>
+    <origin xyz="0.275 0 0.177" rpy="0 0 ${radians(180)}"/>
   </xacro:lidar>
 </robot>

Commit message: Update: LiDARの取り付け角度を変更
ケーブルの引き出し方向を変えたのでそれに伴ってLiDARの角度を変更した

File: adamr2_description/urdf/robot.xacro (robot description, xacro)
@@ -38,5 +38,5 @@
   <!-- lidar -->
   <xacro:lidar parent="base_link">
-    <origin xyz="0.275 0 0.177" rpy="0 0 ${radians(180)}"/>
+    <origin xyz="0.275 0 0.177" rpy="0 0 ${radians(270)}"/>
   </xacro:lidar>
 </robot>

Commit message: Update: Realsenseのリンクを追加

File: adamr2_description/urdf/robot.xacro (robot description, xacro)
@@ -6,4 +6,5 @@
   <xacro:include filename="$(find adamr2_description)/urdf/caster/caster.xacro"/>
   <xacro:include filename="$(find adamr2_description)/urdf/lidar/lidar.xacro"/>
+  <xacro:include filename="$(find adamr2_description)/urdf/camera/camera.xacro"/>
   <!-- base_footprint -->
   <link name="base_footprint"/>
@@ -40,3 +41,7 @@
     <origin xyz="0.275 0 0.177" rpy="0 0 ${radians(270)}"/>
   </xacro:lidar>
+  <!-- camera -->
+  <xacro:camera parent="base_link">
+    <origin xyz="0.280 0.0 0.0625"/>
+  </xacro:camera>
 </robot>
