Commit message: Update: ロボットのハードウェアのモデル

File: adamr2_description/urdf/base/base.xacro (robot description, xacro)
@@ -11,5 +11,5 @@
         <origin xyz="0.0 0.0 0.0"/>
         <geometry>
-          <box size="0.59 0.32 0.275"/>
+          <mesh filename="package://adamr2_description/meshes/base.stl"/>
         </geometry>
         <material name="red">

File: adamr2_description/urdf/caster/caster.xacro (robot description, xacro)
@@ -12,5 +12,5 @@
         <origin rpy="0.0 0.0 0.0"/>
         <geometry>
-          <mesh filename="package://nitic_description/meshes/Caster.STL"/>
+          <mesh filename="package://adamr2_description/meshes/caster.stl"/>
         </geometry>
         <material name="red">

File: adamr2_description/urdf/robot.xacro (robot description, xacro)
@@ -2,3 +2,33 @@
 <robot name="adamr2" xmlns:xacro="http://ros.org/wiki/xacro">
   <xacro:include filename="$(find adamr2_description)/urdf/base/base.xacro"/>
+  <xacro:include filename="$(find adamr2_description)/urdf/wheel/wheel.xacro"/>
+  <xacro:include filename="$(find adamr2_description)/urdf/caster/caster.xacro"/>
+  <!-- base_footprint -->
+  <link name="base_footprint"/>
+  <!-- base_link -->
+  <xacro:base parent="base_footprint">
+    <origin xyz="0.0 0.0 0.262"/>
+  </xacro:base>
+  <!--wheels-->
+  <!-- left -->
+  <xacro:wheel prefix="left" parent="base_link">
+    <origin xyz="0.0 0.1915 -184.5"/>
+    <axis xyz="0 1 0"/>
+  </xacro:wheel>
+  <!-- right -->
+  <xacro:wheel prefix="right" parent="base_link">
+    <origin xyz="0.0 -0.1915 -184.5"/>
+    <axis xyz="0 -1 0"/>
+  </xacro:wheel>
+  <!--casters-->
+  <!-- back -->
+  <xacro:caster prefix="back" parent="base_link">
+    <origin xyz="-0.275 0.0 -149.8"/>
+    <axis xyz="0 0 1"/>
+  </xacro:caster>
+  <!-- front -->
+  <xacro:caster prefix="front" parent="base_link">
+    <origin xyz="0.275 0.0 -149.8"/>
+    <axis xyz="0 0 1"/>
+  </xacro:caster>
 </robot>

File: adamr2_description/urdf/wheel/wheel.xacro (robot description, xacro)
@@ -10,6 +10,7 @@
     <link name="${prefix}_wheel_link">
       <visual>
-        <origin rpy="${radians(90)} 0.0 0.0"/>
+        <origin rpy="0.0 0.0 0.0"/>
         <geometry>
+          <mesh filename="package://adamr2_description/meshes/wheel.str"/>
         </geometry>
         <material name="black">

Commit message: Fix: 参照STLファイルの名前を間違えていたのを修正

File: adamr2_description/urdf/base/base.xacro (robot description, xacro)
@@ -11,5 +11,5 @@
         <origin xyz="0.0 0.0 0.0"/>
         <geometry>
-          <mesh filename="package://adamr2_description/meshes/base.stl"/>
+          <mesh filename="package://adamr2_description/meshes/base_link.STL"/>
         </geometry>
         <material name="red">

File: adamr2_description/urdf/caster/caster.xacro (robot description, xacro)
@@ -12,5 +12,5 @@
         <origin rpy="0.0 0.0 0.0"/>
         <geometry>
-          <mesh filename="package://adamr2_description/meshes/caster.stl"/>
+          <mesh filename="package://adamr2_description/meshes/caster_link.STL"/>
         </geometry>
         <material name="red">

File: adamr2_description/urdf/wheel/wheel.xacro (robot description, xacro)
@@ -12,5 +12,5 @@
         <origin rpy="0.0 0.0 0.0"/>
         <geometry>
-          <mesh filename="package://adamr2_description/meshes/wheel.str"/>
+          <mesh filename="package://adamr2_description/meshes/wheel_link.STL"/>
         </geometry>
         <material name="black">

Commit message: Fix: 慣性モーメント行列を正しい値に修正

File: adamr2_description/urdf/base/base.xacro (robot description, xacro)
@@ -18,7 +18,7 @@
       </visual>
       <inertial>
-        <origin xyz="0.0 0.0 0.0"/>
-        <mass value="22.68"/>
-        <inertia ixx="0.39" ixy="0.04" ixz="0.0" iyy="0.64" iyz="0.02" izz="0.70"/>
+        <origin xyz="-0.02926 0.0 -0.05722"/>
+        <mass value="23.67"/>
+        <inertia ixx="0.43649" ixy="7.4638e-6" ixz="0.03632" iyy="0.73647" iyz="-8.65696e-6" izz="0.66577"/>
       </inertial>
       <collision>
