Commit message: Update: ホイールの当たり判定にSTLファイルをそのまま使うように変更

File: adamr2_description/urdf/wheel/wheel.xacro (robot description, xacro)
@@ -24,7 +24,7 @@
       </inertial>
       <collision>
-        <origin xyz="0.0 0.0 0.0" rpy="${radians(90)} 0.0 0.0"/>
+        <origin xyz="0.0 0.0 0.0"/>
         <geometry>
-          <cylinder radius="0.0775" length="0.030"/>
+          <mesh filename="package://adamr2_description/meshes/wheel_link.STL"/>
         </geometry>
       </collision>

Commit message: Update: 慣性モーメントの値をより詳細な値に変更

File: adamr2_description/urdf/wheel/wheel.xacro (robot description, xacro)
@@ -21,5 +21,5 @@
         <origin xyz="0.0 0.0 0.0"/>
         <mass value="0.4"/>
-        <inertia ixx="0.001" ixy="0.0" ixz="0.0" iyy="0.0006" iyz="0.0" izz="0.0006"/>
+        <inertia ixx="6.56249e-4" ixy="0.0" ixz="0.0" iyy="1.26131e-3" iyz="0.0" izz="6.56249e-4"/>
       </inertial>
       <collision>

Commit message: Update: 車輪の当たり判定をプリミティブ図形に変更

File: adamr2_description/urdf/wheel/wheel.xacro (robot description, xacro)
@@ -24,7 +24,7 @@
       </inertial>
       <collision>
-        <origin xyz="0.0 0.0 0.0"/>
+        <origin xyz="0.0 0.0 0.0" rpy="${radians(90)} 0.0 0.0"/>
         <geometry>
-          <mesh filename="package://adamr2_description/meshes/wheel_link.STL"/>
+          <cylinder radius="0.0775" length="0.030"/>
         </geometry>
       </collision>
