Commit message: Fix: 不要な要素を削除
actuator要素のhardwareInterfaceはIndigoから削除されていた！

File: adamr2_description/urdf/wheel/transmission.xacro (robot description, xacro)
@@ -1,5 +1,5 @@
 <?xml version="1.0"?>
 <robot xmlns:xacro="http://ros.org/wiki/xacro">
-	<xacro:macro name="wheel_trans" params="prefix">
+  <xacro:macro name="wheel_trans" params="prefix">
     <transmission name="${prefix}_wheel_trans">
       <type>transmission_interface/SimpleTransmission</type>
@@ -8,5 +8,4 @@
       </joint>
       <actuator name="${prefix}_wheel_motor">
-        <hardwareInterface>hardware_interface/VelocityJointInterface</hardwareInterface>
         <mechanicalReduction>1</mechanicalReduction>
       </actuator>
