Commit message: Update: キャスターの各リンクの重心と慣性モーメントを適切なものに変更

File: adamr2_description/urdf/caster/caster.xacro (robot description, xacro)
@@ -19,7 +19,7 @@
       </visual>
       <inertial>
-        <origin xyz="0.0 0.0 0.0"/>
+        <origin xyz="6.7e-4 0.0 -0.02699"/>
         <mass value="0.3"/>
-        <inertia ixx="1e-5" ixy="0.0" ixz="0.0" iyy="1e-5" iyz="0.0" izz="1e-5"/>
+        <inertia ixx="4.6263e-4" ixy="-2.12e-9" ixz="5.9561e-5" iyy="5.145e-4" iyz="7.11e-9" izz="2.0407e-4"/>
       </inertial>
     </link>
@@ -34,5 +34,5 @@
         <origin xyz="0.0 0.0 0.0"/>
         <mass value="0.17"/>
-        <inertia ixx="1e-5" ixy="0.0" ixz="0.0" iyy="1e-5" iyz="0.0" izz="1e-5"/>
+        <inertia ixx="6.9281e-5" ixy="0.0" ixz="0.0" iyy="1.0773e-4" iyz="0.0" izz="6.9281e-5"/>
       </inertial>
       <collision>

Commit message: Update: リンクの見た目を更新

File: adamr2_description/urdf/caster/caster.xacro (robot description, xacro)
@@ -12,5 +12,5 @@
         <origin rpy="0.0 0.0 0.0"/>
         <geometry>
-          <mesh filename="package://adamr2_description/meshes/caster_link.STL"/>
+          <mesh filename="package://adamr2_description/meshes/caster_support_link.STL"/>
         </geometry>
         <material name="red">
@@ -31,4 +31,13 @@
     </joint>
     <link name="${prefix}_caster_wheel_link">
+      <visual>
+        <origin rpy="0.0 0.0 0.0"/>
+        <geometry>
+          <mesh filename="package://adamr2_description/meshes/caster_wheel_link.STL"/>
+        </geometry>
+        <material name="red">
+          <color rgba="0.0 0.0 0.0 1.0"/>
+        </material>
+      </visual>
       <inertial>
         <origin xyz="0.0 0.0 0.0"/>

Commit message: Update: 実機用のキャスターリンクURDFファイル
実機ではcontinuousジョイントを使っても回転量がわからないのでTFのエラーが出る，なのでfixedジョイントを使う

File: adamr2_description/urdf/caster/caster.xacro (robot description, xacro)
@@ -2,5 +2,5 @@
 <robot xmlns:xacro="http://ros.org/wiki/xacro">
   <xacro:macro name="caster" params="prefix parent *joint_origin *joint_axis">
-    <joint name="${prefix}_caster_support_joint" type="continuous">
+    <joint name="${prefix}_caster_support_joint" type="fixed">
       <xacro:insert_block name="joint_origin"/>
       <parent link="${parent}"/>
@@ -24,5 +24,5 @@
       </inertial>
     </link>
-    <joint name="${prefix}_caster_wheel_joint" type="continuous">
+    <joint name="${prefix}_caster_wheel_joint" type="fixed">
       <origin xyz="-0.030 0.0 -0.072" rpy="0.0 0.0 0.0"/>
       <parent link="${prefix}_caster_support_link"/>

Commit message: Update: 余計なエレメントを削除
実機用のキャスターリンクジョイントは固定なのでジョイント軸の設定は必要ない

File: adamr2_description/urdf/caster/caster.xacro (robot description, xacro)
@@ -1,10 +1,9 @@
 <?xml version="1.0"?>
 <robot xmlns:xacro="http://ros.org/wiki/xacro">
-  <xacro:macro name="caster" params="prefix parent *joint_origin *joint_axis">
+  <xacro:macro name="caster" params="prefix parent *joint_origin">
     <joint name="${prefix}_caster_support_joint" type="fixed">
       <xacro:insert_block name="joint_origin"/>
       <parent link="${parent}"/>
       <child link="${prefix}_caster_support_link"/>
-      <xacro:insert_block name="joint_axis"/>
     </joint>
     <link name="${prefix}_caster_support_link">
@@ -28,5 +27,4 @@
       <parent link="${prefix}_caster_support_link"/>
       <child link="${prefix}_caster_wheel_link"/>
-      <axis xyz="0.0 1 0.0"/>
     </joint>
     <link name="${prefix}_caster_wheel_link">

File: adamr2_description/urdf/robot.xacro (robot description, xacro)
@@ -30,10 +30,8 @@
   <xacro:caster prefix="back" parent="base_link">
     <origin xyz="-0.275 0.0 -0.1498"/>
-    <axis xyz="0 0 1"/>
   </xacro:caster>
   <!-- front -->
   <xacro:caster prefix="front" parent="base_link">
     <origin xyz="0.275 0.0 -0.1498" rpy="0 0 ${radians(180)}"/>
-    <axis xyz="0 0 1"/>
   </xacro:caster>
   <!-- lidar -->
