Commit message: Update: LiDARリンクを追加

File: adamr2_description/urdf/lidar/lidar.xacro (robot description, xacro)
@@ -1,14 +1,14 @@
 <?xml version="1.0"?>
 <robot xmlns:xacro="http://ros.org/wiki/xacro">
-  <xacro:macro name="lrf" params="prefix parent *joint_origin">
-    <joint name="${prefix}_lrf_joint" type="fixed">
+  <xacro:macro name="lidar" params="parent *joint_origin">
+    <joint name="lidar_joint" type="fixed">
       <xacro:insert_block name="joint_origin"/>
       <parent link="${parent}"/>
-      <child link="${prefix}_lrf_link"/>
+      <child link="lidar_link"/>
     </joint>
-    <link name="${prefix}_lrf_link">
+    <link name="lidar_link">
       <visual>
         <geometry>
-          <mesh filename="package://nitic_description/meshes/LRF.STL"/>
+          <mesh filename="package://adamr2_description/meshes/lidar_link.STL"/>
         </geometry>
         <material name="blue">

File: adamr2_description/urdf/robot.xacro (robot description, xacro)
@@ -4,4 +4,5 @@
   <xacro:include filename="$(find adamr2_description)/urdf/wheel/wheel.xacro"/>
   <xacro:include filename="$(find adamr2_description)/urdf/caster/caster.xacro"/>
+  <xacro:include filename="$(find adamr2_description)/urdf/lidar/lidar.xacro"/>
   <!-- base_footprint -->
   <link name="base_footprint"/>
@@ -32,3 +33,7 @@
     <axis xyz="0 0 1"/>
   </xacro:caster>
+  <!-- lidar -->
+  <xacro:lidar parent="base_link">
+    <origin xyz="0.275 0 0.177"/>
+  </xacro:lidar>
 </robot>

Commit message: Update: lidar_link macro
モデルの見た目の向きを独立して変更出来るようにした

File: adamr2_description/urdf/lidar/lidar.xacro (robot description, xacro)
@@ -1,5 +1,5 @@
 <?xml version="1.0"?>
 <robot xmlns:xacro="http://ros.org/wiki/xacro">
-  <xacro:macro name="lidar" params="parent *joint_origin">
+  <xacro:macro name="lidar" params="parent visual_yaw_orientation *joint_origin">
     <joint name="lidar_joint" type="fixed">
       <xacro:insert_block name="joint_origin"/>
@@ -9,4 +9,5 @@
     <link name="lidar_link">
       <visual>
+        <origin xyz="0.0 0.0 0.0" rpy="0 0 ${visual_yaw_orientation}"/>
         <geometry>
           <mesh filename="package://adamr2_description/meshes/lidar_link.STL"/>

File: adamr2_description/urdf/robot.xacro (robot description, xacro)
@@ -36,5 +36,5 @@
   </xacro:caster>
   <!-- lidar -->
-  <xacro:lidar parent="base_link">
+  <xacro:lidar parent="base_link" visual_yaw_orientation="${radians(180)}">
     <origin xyz="0.275 0 0.177" rpy="0 0 ${radians(270)}"/>
   </xacro:lidar>

File: adamr2_description/urdf/robot_sim.xacro (robot description, xacro)
@@ -46,5 +46,5 @@
   <xacro:caster_gazebo prefix="front"/>
   <!-- lidar -->
-  <xacro:lidar parent="base_link">
+  <xacro:lidar parent="base_link" visual_yaw_orientation="${radians(0)}">
     <origin xyz="0.275 0 0.177" rpy="0 0 0"/>
   </xacro:lidar>
